File: eagle/VA-Meter.brd (EAGLE design)
At the start: 100 x 80 mm, 23 parts, among them IC1 MEGA328P, IC2 7805TV

Commit message: 回路図を修正　シャントレギュレータの接続
Connections:
- net GND: now also VR1.R
- net V-: no longer VR1.R
Changed lines of the file:
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@@
 <contactref element="VR1" pad="C"/>
 <contactref element="GND" pad="3"/>
-<wire x1="-19.05" y1="60.96" x2="-24.13" y2="66.04" width="0" layer="19" extent="1-1"/>
+<contactref element="VR1" pad="R"/>
+<wire x1="-21.59" y1="60.96" x2="-24.13" y2="66.04" width="0" layer="19" extent="1-1"/>
+<wire x1="-19.05" y1="60.96" x2="-21.59" y2="60.96" width="0" layer="19" extent="1-1"/>
 <wire x1="-34.29" y1="66.04" x2="-24.13" y2="66.04" width="0" layer="19" extent="1-1"/>
-<wire x1="-29.21" y1="39.37" x2="-19.05" y2="60.96" width="0" layer="19" extent="1-1"/>
+<wire x1="-29.21" y1="39.37" x2="-21.59" y2="60.96" width="0" layer="19" extent="1-1"/>
 <wire x1="-46.99" y1="39.37" x2="-29.21" y2="39.37" width="0" layer="19" extent="1-1"/>
 <wire x1="-16.51" y1="6.985" x2="-29.21" y2="39.37" width="0" layer="19" extent="1-1"/>
@@
 <contactref element="R8" pad="2"/>
 <contactref element="IC2" pad="2"/>
-<contactref element="VR1" pad="R"/>
 <contactref element="C2" pad="-"/>
 <contactref element="C3" pad="-"/>
@@
 <wire x1="-44.45" y1="46.99" x2="-45.72" y2="54.61" width="0" layer="19" extent="1-1"/>
 <wire x1="-44.45" y1="66.04" x2="-45.72" y2="54.61" width="0" layer="19" extent="1-1"/>
-<wire x1="-21.59" y1="60.96" x2="-38.1" y2="54.61" width="0" layer="19" extent="1-1"/>
-<wire x1="-20.32" y1="62.865" x2="-21.59" y2="60.96" width="0" layer="19" extent="1-1"/>
-<wire x1="-13.97" y1="46.99" x2="-21.59" y2="60.96" width="0" layer="19" extent="1-1"/>
+<wire x1="-20.32" y1="62.865" x2="-38.1" y2="54.61" width="0" layer="19" extent="1-1"/>
+<wire x1="-13.97" y1="46.99" x2="-20.32" y2="62.865" width="0" layer="19" extent="1-1"/>
 </signal>
 <signal name="V+">

Commit message: 回路図修正
Parts:
- added R11: 1k, rcl:P0613/15
- D1: value 1N4004 -> 1S2; device diode:DO41-10 -> diode:CB417-15
- R8: value 220 -> 3.3k
- moved D1 15.7 mm to (-59.7, -33.0)
Connections:
- new net N$1: R11.1
- net -12V: now also R11.2
Changed lines of the file:
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@@
 <element name="IC2" library="linear" package="TO220V" value="7805TV" x="-29.21" y="34.29"/>
 <element name="VR1" library="v-reg" package="TO92-CLP" value="" x="-20.32" y="60.96"/>
-<element name="R8" library="rcl" package="P0613/15" value="220" x="-21.59" y="46.99"/>
+<element name="R8" library="rcl" package="P0613/15" value="3.3k" x="-21.59" y="46.99"/>
 <element name="GND" library="con-wago-508" package="W237-133" value="" x="-21.59" y="7.62">
 <attribute name="OC_NEWARK" value="unknown" x="0" y="0" size="1.778" layer="27" display="off"/>
@@
 </element>
 <element name="JP2" library="pinhead" package="1X02" value="" x="-66.04" y="-11.43"/>
-<element name="D1" library="diode" package="DO41-10" value="1N4004" x="-63.5" y="-17.78"/>
+<element name="R11" library="rcl" package="P0613/15" value="1k" x="-60.96" y="-26.67"/>
+<element name="D1" library="diode" package="CB417-15" value="1S2" x="-59.69" y="-33.02"/>
 </elements>
 <signals>
@@
 <contactref element="V-IN" pad="1"/>
 <contactref element="D1" pad="C"/>
-<wire x1="-67.31" y1="0.635" x2="-68.58" y2="-17.78" width="0" layer="19" extent="1-1"/>
+<wire x1="-67.31" y1="0.635" x2="-67.31" y2="-33.02" width="0" layer="19" extent="1-1"/>
 <wire x1="-31.75" y1="31.75" x2="-67.31" y2="0.635" width="0" layer="19" extent="1-1"/>
 <wire x1="-46.99" y1="46.99" x2="-31.75" y2="31.75" width="0" layer="19" extent="1-1"/>
@@
 <contactref element="R7" pad="A"/>
 <contactref element="D1" pad="A"/>
-<wire x1="-57.15" y1="-3.81" x2="-58.42" y2="-17.78" width="0" layer="19" extent="1-1"/>
+<wire x1="-57.15" y1="-3.81" x2="-52.07" y2="-33.02" width="0" layer="19" extent="1-1"/>
 <wire x1="-33.02" y1="15.24" x2="-57.15" y2="-3.81" width="0" layer="19" extent="1-1"/>
 <wire x1="-41.91" y1="29.21" x2="-33.02" y2="15.24" width="0" layer="19" extent="1-1"/>
@@
 <contactref element="R8" pad="1"/>
 <contactref element="V-IN" pad="2"/>
+<contactref element="R11" pad="2"/>
+<wire x1="-62.23" y1="0.635" x2="-53.34" y2="-26.67" width="0" layer="19" extent="1-1"/>
 <wire x1="-29.21" y1="46.99" x2="-62.23" y2="0.635" width="0" layer="19" extent="1-1"/>
 </signal>
@@
 <wire x1="-31.75" y1="59.69" x2="-64.77" y2="-11.43" width="0" layer="19" extent="1-1"/>
 </signal>
+<signal name="N$1">
+<contactref element="R11" pad="1"/>
+</signal>
 </signals>
