File: eagle/VA-Meter-I2C.brd (EAGLE design)
At the start: 100 x 80 mm, 21 parts, among them IC1 MEGA328P, IC2 7805TV

Commit message: I2C-LCD 回路図を修正
Parts:
- removed R11: 1k, rcl:P0613/15
- added D2: 3.3V, diode:ZDIO-5
- added JP3: LCD-BL, pinhead:1X02
- added R12: 1.5k, rcl:0207/7
- added R13: 1k, rcl:0207/7
- added R2: 220, rcl:0207/7
- added R4: 470, rcl:0207/7
- added R7: 1.2k, rcl:0207/7
- added VR2: (no value), v-reg:TO92-CLP
- R8: value 3.3k -> 100
Connections:
- removed net N$1: R11.1
- removed net N$16: C1.1, IC1.20, L1.1
- new net +3V3: D2.C, JP1.1, R2.1
- new net N$5: C1.1, IC1.20, L1.1, R13.2
- new net N$6: R12.2, R7.1, VR2.R
- new net N$7: IC1.21, R13.1, R7.2, VR2.C
- net -12V: no longer R11.2
- net N$2: now also JP3.2, R4.1; no longer JP1.4
- net V+: now also R2.2, R4.2; no longer JP1.1
- net V-: now also D2.A, JP1.4, JP3.1, R12.1, VR2.A
Changed lines of the file:
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@@
 <element name="IC2" library="linear" package="TO220V" value="7805TV" x="-29.21" y="34.29"/>
 <element name="VR1" library="v-reg" package="TO92-CLP" value="" x="-20.32" y="60.96"/>
-<element name="R8" library="rcl" package="P0613/15" value="3.3k" x="-21.59" y="46.99"/>
+<element name="R8" library="rcl" package="P0613/15" value="100" x="-21.59" y="46.99"/>
 <element name="GND" library="con-wago-508" package="W237-133" value="" x="-21.59" y="7.62">
 <attribute name="OC_NEWARK" value="unknown" x="0" y="0" size="1.778" layer="27" display="off"/>
@@
 </element>
 <element name="JP2" library="pinhead" package="1X02" value="" x="-66.04" y="-11.43"/>
-<element name="R11" library="rcl" package="P0613/15" value="1k" x="-60.96" y="-26.67"/>
 <element name="D1" library="diode" package="CB417-15" value="1S2" x="-59.69" y="-33.02"/>
 <element name="JP1" library="pinhead" package="1X07" value="I2C-LCD" x="-59.69" y="-39.37"/>
+<element name="D2" library="diode" package="ZDIO-5" value="3.3V" x="-66.04" y="-46.99"/>
+<element name="R2" library="rcl" package="0207/7" value="220" x="-64.77" y="-52.07"/>
+<element name="JP3" library="pinhead" package="1X02" value="LCD-BL" x="-66.04" y="-57.15"/>
+<element name="R4" library="rcl" package="0207/7" value="470" x="-64.77" y="-64.77"/>
+<element name="VR2" library="v-reg" package="TO92-CLP" value="" x="-66.04" y="-69.85"/>
+<element name="R7" library="rcl" package="0207/7" value="1.2k" x="-64.77" y="-74.93"/>
+<element name="R12" library="rcl" package="0207/7" value="1.5k" x="-64.77" y="-80.01"/>
+<element name="R13" library="rcl" package="0207/7" value="1k" x="-64.77" y="-85.09"/>
 </elements>
 <signals>
@@
 <contactref element="IC1" pad="8"/>
 <contactref element="C4" pad="2"/>
+<contactref element="D2" pad="A"/>
+<contactref element="JP1" pad="4"/>
+<contactref element="JP3" pad="1"/>
+<contactref element="VR2" pad="A"/>
+<contactref element="R12" pad="1"/>
+<wire x1="-66.04" y1="-67.945" x2="-68.58" y2="-80.01" width="0" layer="19" extent="1-1"/>
+<wire x1="-67.31" y1="-57.15" x2="-66.04" y2="-67.945" width="0" layer="19" extent="1-1"/>
+<wire x1="-63.5" y1="-46.99" x2="-67.31" y2="-57.15" width="0" layer="19" extent="1-1"/>
+<wire x1="-59.69" y1="-39.37" x2="-63.5" y2="-46.99" width="0" layer="19" extent="1-1"/>
+<wire x1="-52.07" y1="-3.81" x2="-59.69" y2="-39.37" width="0" layer="19" extent="1-1"/>
 <wire x1="-30.48" y1="15.24" x2="-52.07" y2="-3.81" width="0" layer="19" extent="1-1"/>
 <wire x1="-33.02" y1="22.86" x2="-30.48" y2="15.24" width="0" layer="19" extent="1-1"/>
@@
 <contactref element="C4" pad="1"/>
 <contactref element="D1" pad="A"/>
-<contactref element="JP1" pad="1"/>
-<wire x1="-52.07" y1="-33.02" x2="-67.31" y2="-39.37" width="0" layer="19" extent="1-1"/>
+<contactref element="R2" pad="2"/>
+<contactref element="R4" pad="2"/>
+<wire x1="-60.96" y1="-52.07" x2="-60.96" y2="-64.77" width="0" layer="19" extent="1-1"/>
+<wire x1="-52.07" y1="-33.02" x2="-60.96" y2="-52.07" width="0" layer="19" extent="1-1"/>
 <wire x1="-57.15" y1="-3.81" x2="-52.07" y2="-33.02" width="0" layer="19" extent="1-1"/>
 <wire x1="-33.02" y1="15.24" x2="-57.15" y2="-3.81" width="0" layer="19" extent="1-1"/>
@@
 <wire x1="-38.1" y1="46.99" x2="-26.67" y2="31.75" width="0" layer="19" extent="1-1"/>
 </signal>
-<signal name="N$16">
-<contactref element="IC1" pad="20"/>
-<contactref element="C1" pad="1"/>
-<contactref element="L1" pad="1"/>
-<wire x1="-20.28" y1="30.48" x2="-49.53" y2="66.04" width="0" layer="19" extent="1-1"/>
-<wire x1="-27.94" y1="22.86" x2="-20.28" y2="30.48" width="0" layer="19" extent="1-1"/>
-</signal>
 <signal name="-12V">
 <contactref element="R8" pad="1"/>
 <contactref element="V-IN" pad="2"/>
-<contactref element="R11" pad="2"/>
-<wire x1="-62.23" y1="0.635" x2="-53.34" y2="-26.67" width="0" layer="19" extent="1-1"/>
 <wire x1="-29.21" y1="46.99" x2="-62.23" y2="0.635" width="0" layer="19" extent="1-1"/>
 </signal>
@@
 <contactref element="JP2" pad="2"/>
 <wire x1="-31.75" y1="59.69" x2="-64.77" y2="-11.43" width="0" layer="19" extent="1-1"/>
-</signal>
-<signal name="N$1">
-<contactref element="R11" pad="1"/>
-</signal>
-<signal name="N$2">
-<contactref element="JP1" pad="4"/>
 </signal>
 <signal name="SCL">
@@
 <wire x1="-45.72" y1="15.24" x2="-52.07" y2="-39.37" width="0" layer="19" extent="1-1"/>
 </signal>
+<signal name="+3V3">
+<contactref element="R2" pad="1"/>
+<contactref element="D2" pad="C"/>
+<contactref element="JP1" pad="1"/>
+<wire x1="-68.58" y1="-46.99" x2="-68.58" y2="-52.07" width="0" layer="19" extent="1-1"/>
+<wire x1="-67.31" y1="-39.37" x2="-68.58" y2="-46.99" width="0" layer="19" extent="1-1"/>
+</signal>
+<signal name="N$2">
+<contactref element="JP3" pad="2"/>
+<contactref element="R4" pad="1"/>
+<wire x1="-64.77" y1="-57.15" x2="-68.58" y2="-64.77" width="0" layer="19" extent="1-1"/>
+</signal>
+<signal name="N$6">
+<contactref element="VR2" pad="R"/>
+<contactref element="R7" pad="1"/>
+<contactref element="R12" pad="2"/>
+<wire x1="-67.31" y1="-69.85" x2="-68.58" y2="-74.93" width="0" layer="19" extent="1-1"/>
+<wire x1="-60.96" y1="-80.01" x2="-68.58" y2="-74.93" width="0" layer="19" extent="1-1"/>
+</signal>
+<signal name="N$7">
+<contactref element="VR2" pad="C"/>
+<contactref element="R13" pad="1"/>
+<contactref element="R7" pad="2"/>
+<contactref element="IC1" pad="21"/>
+<wire x1="-60.96" y1="-74.93" x2="-68.58" y2="-85.09" width="0" layer="19" extent="1-1"/>
+<wire x1="-64.77" y1="-69.85" x2="-60.96" y2="-74.93" width="0" layer="19" extent="1-1"/>
+<wire x1="-30.48" y1="22.86" x2="-64.77" y2="-69.85" width="0" layer="19" extent="1-1"/>
+</signal>
+<signal name="N$5">
+<contactref element="C1" pad="1"/>
+<contactref element="L1" pad="1"/>
+<contactref element="R13" pad="2"/>
+<contactref element="IC1" pad="20"/>
+<wire x1="-27.94" y1="22.86" x2="-60.96" y2="-85.09" width="0" layer="19" extent="1-1"/>
+<wire x1="-20.28" y1="30.48" x2="-27.94" y2="22.86" width="0" layer="19" extent="1-1"/>
+<wire x1="-49.53" y1="66.04" x2="-20.28" y2="30.48" width="0" layer="19" extent="1-1"/>
+</signal>
 </signals>

Commit message: V-Meter-I2C 回路図修正 シャントレギュレータ－ではなくAVCCを基準電圧に
Parts:
- removed R12: 1.5k, rcl:0207/7
- removed R13: 1k, rcl:0207/7
- removed R7: 1.2k, rcl:0207/7
- removed VR2: (no value), v-reg:TO92-CLP
- added C5, C6, C7: 0.1u, rcl:C050-024X044
Connections:
- net -12V renamed -15V
- removed net +12V: C2.+, D1.C, IC2.1, V-IN.1
- removed net N$5: C1.1, IC1.20, L1.1, R13.2
- removed net N$6: R12.2, R7.1, VR2.R
- removed net N$7: IC1.21, R13.1, R7.2, VR2.C
- new net +15V: C2.+, C6.2, D1.C, IC2.1, V-IN.1
- new net N$10: C1.1, IC1.20, L1.1
- new net N$9: C5.2, IC1.21
- net V+: now also C7.2
- net V-: now also C5.1, C6.1, C7.1; no longer R12.1, VR2.A
Changed lines of the file:
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@@
 <element name="JP3" library="pinhead" package="1X02" value="LCD-BL" x="-66.04" y="-57.15"/>
 <element name="R4" library="rcl" package="0207/7" value="470" x="-64.77" y="-64.77"/>
-<element name="VR2" library="v-reg" package="TO92-CLP" value="" x="-66.04" y="-69.85"/>
-<element name="R7" library="rcl" package="0207/7" value="1.2k" x="-64.77" y="-74.93"/>
-<element name="R12" library="rcl" package="0207/7" value="1.5k" x="-64.77" y="-80.01"/>
-<element name="R13" library="rcl" package="0207/7" value="1k" x="-64.77" y="-85.09"/>
+<element name="C5" library="rcl" package="C050-024X044" value="0.1u" x="-66.04" y="-69.85"/>
+<element name="C6" library="rcl" package="C050-024X044" value="0.1u" x="-66.04" y="-76.2"/>
+<element name="C7" library="rcl" package="C050-024X044" value="0.1u" x="-66.04" y="-82.55"/>
 </elements>
 <signals>
@@
 <wire x1="-16.51" y1="6.985" x2="-29.21" y2="39.37" width="0" layer="19" extent="1-1"/>
 </signal>
-<signal name="+12V">
+<signal name="+15V">
 <contactref element="IC2" pad="1"/>
-<contactref element="C2" pad="+"/>
 <contactref element="V-IN" pad="1"/>
 <contactref element="D1" pad="C"/>
+<contactref element="C2" pad="+"/>
+<contactref element="C6" pad="2"/>
+<wire x1="-67.31" y1="-33.02" x2="-63.5" y2="-76.2" width="0" layer="19" extent="1-1"/>
 <wire x1="-67.31" y1="0.635" x2="-67.31" y2="-33.02" width="0" layer="19" extent="1-1"/>
 <wire x1="-31.75" y1="31.75" x2="-67.31" y2="0.635" width="0" layer="19" extent="1-1"/>
@@
 <contactref element="R8" pad="2"/>
 <contactref element="IC2" pad="2"/>
-<contactref element="C2" pad="-"/>
 <contactref element="C3" pad="-"/>
 <contactref element="IC1" pad="8"/>
@@
 <contactref element="JP1" pad="4"/>
 <contactref element="JP3" pad="1"/>
-<contactref element="VR2" pad="A"/>
-<contactref element="R12" pad="1"/>
-<wire x1="-66.04" y1="-67.945" x2="-68.58" y2="-80.01" width="0" layer="19" extent="1-1"/>
-<wire x1="-67.31" y1="-57.15" x2="-66.04" y2="-67.945" width="0" layer="19" extent="1-1"/>
+<contactref element="C5" pad="1"/>
+<contactref element="C2" pad="-"/>
+<contactref element="C6" pad="1"/>
+<contactref element="C7" pad="1"/>
+<wire x1="-68.58" y1="-76.2" x2="-68.58" y2="-82.55" width="0" layer="19" extent="1-1"/>
+<wire x1="-68.58" y1="-69.85" x2="-68.58" y2="-76.2" width="0" layer="19" extent="1-1"/>
+<wire x1="-67.31" y1="-57.15" x2="-68.58" y2="-69.85" width="0" layer="19" extent="1-1"/>
 <wire x1="-63.5" y1="-46.99" x2="-67.31" y2="-57.15" width="0" layer="19" extent="1-1"/>
 <wire x1="-59.69" y1="-39.37" x2="-63.5" y2="-46.99" width="0" layer="19" extent="1-1"/>
@@
 <contactref element="R2" pad="2"/>
 <contactref element="R4" pad="2"/>
+<contactref element="C7" pad="2"/>
+<wire x1="-60.96" y1="-64.77" x2="-63.5" y2="-82.55" width="0" layer="19" extent="1-1"/>
 <wire x1="-60.96" y1="-52.07" x2="-60.96" y2="-64.77" width="0" layer="19" extent="1-1"/>
 <wire x1="-52.07" y1="-33.02" x2="-60.96" y2="-52.07" width="0" layer="19" extent="1-1"/>
@@
 <wire x1="-38.1" y1="46.99" x2="-26.67" y2="31.75" width="0" layer="19" extent="1-1"/>
 </signal>
-<signal name="-12V">
+<signal name="-15V">
 <contactref element="R8" pad="1"/>
 <contactref element="V-IN" pad="2"/>
@@
 <wire x1="-64.77" y1="-57.15" x2="-68.58" y2="-64.77" width="0" layer="19" extent="1-1"/>
 </signal>
-<signal name="N$6">
-<contactref element="VR2" pad="R"/>
-<contactref element="R7" pad="1"/>
-<contactref element="R12" pad="2"/>
-<wire x1="-67.31" y1="-69.85" x2="-68.58" y2="-74.93" width="0" layer="19" extent="1-1"/>
-<wire x1="-60.96" y1="-80.01" x2="-68.58" y2="-74.93" width="0" layer="19" extent="1-1"/>
+<signal name="N$9">
+<contactref element="IC1" pad="21"/>
+<contactref element="C5" pad="2"/>
+<wire x1="-30.48" y1="22.86" x2="-63.5" y2="-69.85" width="0" layer="19" extent="1-1"/>
 </signal>
-<signal name="N$7">
-<contactref element="VR2" pad="C"/>
-<contactref element="R13" pad="1"/>
-<contactref element="R7" pad="2"/>
-<contactref element="IC1" pad="21"/>
-<wire x1="-60.96" y1="-74.93" x2="-68.58" y2="-85.09" width="0" layer="19" extent="1-1"/>
-<wire x1="-64.77" y1="-69.85" x2="-60.96" y2="-74.93" width="0" layer="19" extent="1-1"/>
-<wire x1="-30.48" y1="22.86" x2="-64.77" y2="-69.85" width="0" layer="19" extent="1-1"/>
-</signal>
-<signal name="N$5">
+<signal name="N$10">
 <contactref element="C1" pad="1"/>
 <contactref element="L1" pad="1"/>
-<contactref element="R13" pad="2"/>
 <contactref element="IC1" pad="20"/>
-<wire x1="-27.94" y1="22.86" x2="-60.96" y2="-85.09" width="0" layer="19" extent="1-1"/>
-<wire x1="-20.28" y1="30.48" x2="-27.94" y2="22.86" width="0" layer="19" extent="1-1"/>
-<wire x1="-49.53" y1="66.04" x2="-20.28" y2="30.48" width="0" layer="19" extent="1-1"/>
+<wire x1="-20.28" y1="30.48" x2="-49.53" y2="66.04" width="0" layer="19" extent="1-1"/>
+<wire x1="-27.94" y1="22.86" x2="-20.28" y2="30.48" width="0" layer="19" extent="1-1"/>
 </signal>
 </signals>

Commit message: 電源部の保護回路を±のポリスイッチに変更
Parts:
- removed VR1: (no value), v-reg:TO92-CLP
- added C8: 0.1u, rcl:C050-024X044
- added D3: 3.3V, diode:ZDIO-5
- added PF1, PF2: PTC-PF-5.1, polyswitch:PF-5.1
- added R11, R7: 1.5k, rcl:P0613/15
- added T1: 2SA1359, transistor:TO126V
- D2: value 3.3V -> 3.6V
- R8: value 100 -> 1.5k
Connections:
- removed net RESET: IC1.2, JP1.7
- new net N$1: D3.A, R11.2, R7.2, R8.2, T1.2
- new net N$11: IC1.4, JP1.7
- new net N$5: C8.2, T1.3
- new net N$6: PF2.1, V-IN.1
- new net N$7: PF1.1, V-IN.2
- net +15V: now also PF2.2; no longer V-IN.1
- net -15V: now also PF1.2, R11.1, R7.1; no longer V-IN.2
- net GND: now also C8.1, D3.C; no longer VR1.C, VR1.R
- net V-: now also T1.1; no longer R8.2, VR1.A
Changed lines of the file:
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@@
 <layer number="48" name="Document" color="7" fill="1" visible="yes" active="yes"/>
 <layer number="49" name="Reference" color="7" fill="1" visible="yes" active="yes"/>
+<layer number="50" name="dxf" color="7" fill="1" visible="yes" active="yes"/>
 <layer number="51" name="tDocu" color="7" fill="1" visible="yes" active="yes"/>
 <layer number="52" name="bDocu" color="7" fill="1" visible="yes" active="yes"/>
+<layer number="56" name="wert" color="7" fill="1" visible="yes" active="yes"/>
 <layer number="91" name="Nets" color="2" fill="1" visible="no" active="no"/>
 <layer number="92" name="Busses" color="1" fill="1" visible="no" active="no"/>
@@
 <element name="L1" library="rcl" package="6000-XXXX-RC" value="10uH" x="-17.78" y="30.48"/>
 <element name="IC2" library="linear" package="TO220V" value="7805TV" x="-29.21" y="34.29"/>
-<element name="VR1" library="v-reg" package="TO92-CLP" value="" x="-20.32" y="60.96"/>
-<element name="R8" library="rcl" package="P0613/15" value="100" x="-21.59" y="46.99"/>
+<element name="R8" library="rcl" package="P0613/15" value="1.5k" x="-21.59" y="46.99"/>
 <element name="GND" library="con-wago-508" package="W237-133" value="" x="-21.59" y="7.62">
 <attribute name="OC_NEWARK" value="unknown" x="0" y="0" size="1.778" layer="27" display="off"/>
@@
 <element name="D1" library="diode" package="CB417-15" value="1S2" x="-59.69" y="-33.02"/>
 <element name="JP1" library="pinhead" package="1X07" value="I2C-LCD" x="-59.69" y="-39.37"/>
-<element name="D2" library="diode" package="ZDIO-5" value="3.3V" x="-66.04" y="-46.99"/>
+<element name="D2" library="diode" package="ZDIO-5" value="3.6V" x="-66.04" y="-46.99"/>
 <element name="R2" library="rcl" package="0207/7" value="220" x="-64.77" y="-52.07"/>
 <element name="JP3" library="pinhead" package="1X02" value="LCD-BL" x="-66.04" y="-57.15"/>
@@
 <element name="C6" library="rcl" package="C050-024X044" value="0.1u" x="-66.04" y="-76.2"/>
 <element name="C7" library="rcl" package="C050-024X044" value="0.1u" x="-66.04" y="-82.55"/>
+<element name="D3" library="diode" package="ZDIO-5" value="3.3V" x="-66.04" y="-90.17"/>
+<element name="C8" library="rcl" package="C050-024X044" value="0.1u" x="-66.04" y="-97.79"/>
+<element name="T1" library="transistor" package="TO126V" value="2SA1359" x="-64.77" y="-100.33"/>
+<element name="R7" library="rcl" package="P0613/15" value="1.5k" x="-60.96" y="-110.49"/>
+<element name="R11" library="rcl" package="P0613/15" value="1.5k" x="-60.96" y="-118.11"/>
+<element name="PF2" library="polyswitch" package="PF-5.1" value="PTC-PF-5.1" x="-64.77" y="-128.27"/>
+<element name="PF1" library="polyswitch" package="PF-5.1" value="PTC-PF-5.1" x="-64.77" y="-144.78"/>
 </elements>
 <signals>
@@
 <contactref element="R5" pad="1"/>
 <contactref element="R6" pad="1"/>
-<contactref element="VR1" pad="C"/>
 <contactref element="GND" pad="3"/>
-<contactref element="VR1" pad="R"/>
 <contactref element="R10" pad="2"/>
 <contactref element="R9" pad="2"/>
-<wire x1="-21.59" y1="60.96" x2="-19.05" y2="60.96" width="0" layer="19" extent="1-1"/>
-<wire x1="-24.13" y1="66.04" x2="-21.59" y2="60.96" width="0" layer="19" extent="1-1"/>
+<contactref element="D3" pad="C"/>
+<contactref element="C8" pad="1"/>
+<wire x1="-68.58" y1="-90.17" x2="-68.58" y2="-97.79" width="0" layer="19" extent="1-1"/>
+<wire x1="-16.51" y1="6.985" x2="-68.58" y2="-90.17" width="0" layer="19" extent="1-1"/>
+<wire x1="-29.21" y1="39.37" x2="-16.51" y2="6.985" width="0" layer="19" extent="1-1"/>
+<wire x1="-46.99" y1="39.37" x2="-29.21" y2="39.37" width="0" layer="19" extent="1-1"/>
+<wire x1="-24.13" y1="66.04" x2="-29.21" y2="39.37" width="0" layer="19" extent="1-1"/>
 <wire x1="-34.29" y1="66.04" x2="-24.13" y2="66.04" width="0" layer="19" extent="1-1"/>
-<wire x1="-29.21" y1="39.37" x2="-21.59" y2="60.96" width="0" layer="19" extent="1-1"/>
-<wire x1="-46.99" y1="39.37" x2="-29.21" y2="39.37" width="0" layer="19" extent="1-1"/>
-<wire x1="-16.51" y1="6.985" x2="-29.21" y2="39.37" width="0" layer="19" extent="1-1"/>
 </signal>
 <signal name="+15V">
 <contactref element="IC2" pad="1"/>
-<contactref element="V-IN" pad="1"/>
 <contactref element="D1" pad="C"/>
 <contactref element="C2" pad="+"/>
 <contactref element="C6" pad="2"/>
+<contactref element="PF2" pad="2"/>
+<wire x1="-63.5" y1="-76.2" x2="-62.22" y2="-128.27" width="0" layer="19" extent="1-1"/>
 <wire x1="-67.31" y1="-33.02" x2="-63.5" y2="-76.2" width="0" layer="19" extent="1-1"/>
-<wire x1="-67.31" y1="0.635" x2="-67.31" y2="-33.02" width="0" layer="19" extent="1-1"/>
-<wire x1="-31.75" y1="31.75" x2="-67.31" y2="0.635" width="0" layer="19" extent="1-1"/>
+<wire x1="-31.75" y1="31.75" x2="-67.31" y2="-33.02" width="0" layer="19" extent="1-1"/>
 <wire x1="-46.99" y1="46.99" x2="-31.75" y2="31.75" width="0" layer="19" extent="1-1"/>
 </signal>
@@
 <contactref element="IC1" pad="22"/>
 <contactref element="C1" pad="2"/>
-<contactref element="VR1" pad="A"/>
-<contactref element="R8" pad="2"/>
 <contactref element="IC2" pad="2"/>
 <contactref element="C3" pad="-"/>
@@
 <contactref element="C6" pad="1"/>
 <contactref element="C7" pad="1"/>
+<contactref element="T1" pad="1"/>
+<wire x1="-68.58" y1="-82.55" x2="-67.056" y2="-101.6" width="0" layer="19" extent="1-1"/>
 <wire x1="-68.58" y1="-76.2" x2="-68.58" y2="-82.55" width="0" layer="19" extent="1-1"/>
 <wire x1="-68.58" y1="-69.85" x2="-68.58" y2="-76.2" width="0" layer="19" extent="1-1"/>
@@
 <wire x1="-44.45" y1="46.99" x2="-35.56" y2="46.99" width="0" layer="19" extent="1-1"/>
 <wire x1="-44.45" y1="66.04" x2="-44.45" y2="46.99" width="0" layer="19" extent="1-1"/>
-<wire x1="-13.97" y1="46.99" x2="-29.21" y2="31.75" width="0" layer="19" extent="1-1"/>
-<wire x1="-20.32" y1="62.865" x2="-13.97" y2="46.99" width="0" layer="19" extent="1-1"/>
 </signal>
 <signal name="V+">
@@
 <signal name="-15V">
 <contactref element="R8" pad="1"/>
-<contactref element="V-IN" pad="2"/>
-<wire x1="-29.21" y1="46.99" x2="-62.23" y2="0.635" width="0" layer="19" extent="1-1"/>
+<contactref element="R11" pad="1"/>
+<contactref element="R7" pad="1"/>
+<contactref element="PF1" pad="2"/>
+<wire x1="-68.58" y1="-118.11" x2="-62.22" y2="-144.78" width="0" layer="19" extent="1-1"/>
+<wire x1="-68.58" y1="-110.49" x2="-68.58" y2="-118.11" width="0" layer="19" extent="1-1"/>
+<wire x1="-29.21" y1="46.99" x2="-68.58" y2="-110.49" width="0" layer="19" extent="1-1"/>
 </signal>
 <signal name="MEAS+">
@@
 <contactref element="IC1" pad="28"/>
 <wire x1="-48.26" y1="22.86" x2="-54.61" y2="-39.37" width="0" layer="19" extent="1-1"/>
-</signal>
-<signal name="RESET">
-<contactref element="IC1" pad="2"/>
-<contactref element="JP1" pad="7"/>
-<wire x1="-45.72" y1="15.24" x2="-52.07" y2="-39.37" width="0" layer="19" extent="1-1"/>
 </signal>
 <signal name="+3V3">
@@
 <wire x1="-27.94" y1="22.86" x2="-20.28" y2="30.48" width="0" layer="19" extent="1-1"/>
 </signal>
+<signal name="N$1">
+<contactref element="R8" pad="2"/>
+<contactref element="D3" pad="A"/>
+<contactref element="T1" pad="2"/>
+<contactref element="R11" pad="2"/>
+<contactref element="R7" pad="2"/>
+<wire x1="-53.34" y1="-110.49" x2="-53.34" y2="-118.11" width="0" layer="19" extent="1-1"/>
+<wire x1="-64.77" y1="-101.6" x2="-53.34" y2="-110.49" width="0" layer="19" extent="1-1"/>
+<wire x1="-63.5" y1="-90.17" x2="-64.77" y2="-101.6" width="0" layer="19" extent="1-1"/>
+<wire x1="-13.97" y1="46.99" x2="-63.5" y2="-90.17" width="0" layer="19" extent="1-1"/>
+</signal>
+<signal name="N$5">
+<contactref element="T1" pad="3"/>
+<contactref element="C8" pad="2"/>
+<wire x1="-63.5" y1="-97.79" x2="-62.484" y2="-101.6" width="0" layer="19" extent="1-1"/>
+</signal>
+<signal name="N$6">
+<contactref element="V-IN" pad="1"/>
+<contactref element="PF2" pad="1"/>
+<wire x1="-67.31" y1="0.635" x2="-67.32" y2="-128.27" width="0" layer="19" extent="1-1"/>
+</signal>
+<signal name="N$11">
+<contactref element="IC1" pad="4"/>
+<contactref element="JP1" pad="7"/>
+<wire x1="-40.64" y1="15.24" x2="-52.07" y2="-39.37" width="0" layer="19" extent="1-1"/>
+</signal>
+<signal name="N$7">
+<contactref element="V-IN" pad="2"/>
+<contactref element="PF1" pad="1"/>
+<wire x1="-62.23" y1="0.635" x2="-67.32" y2="-144.78" width="0" layer="19" extent="1-1"/>
+</signal>
 </signals>
