File: eagle/VA-Meter_Analog_Part.brd (EAGLE design)
At the start: 100 x 80 mm, 17 parts, among them IC2 LM358N

Commit message: アナログ部の修正 電流値の増幅を11倍に変更
Parts:
- R2, R8: value 2k -> 1k
Changed lines of the file:
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@@
 <?xml version="1.0" encoding="utf-8"?>
 <!DOCTYPE eagle SYSTEM "eagle.dtd">
-<eagle version="6.6.0">
+<eagle version="7.1.0">
 <drawing>
 <settings>
@@
 <pass name="Default">
 <param name="RoutingGrid" value="50mil"/>
+<param name="AutoGrid" value="1"/>
+<param name="Efforts" value="0"/>
+<param name="TopRouterVariant" value="1"/>
 <param name="tpViaShape" value="round"/>
 <param name="PrefDir.1" value="|"/>
@@
 <element name="JP4" library="pinhead" package="1X03" value="Power\" x="60.96" y="17.78" rot="R270"/>
 <element name="IC2" library="linear" package="DIL08" value="LM358N" x="46.99" y="21.59"/>
-<element name="R2" library="rcl" package="0207/7" value="2k" x="45.72" y="11.43" rot="R270"/>
+<element name="R2" library="rcl" package="0207/7" value="1k" x="45.72" y="11.43" rot="R270"/>
 <element name="R7" library="rcl" package="0207/7" value="10k" x="43.18" y="11.43" rot="R90"/>
-<element name="R8" library="rcl" package="0207/7" value="2k" x="48.26" y="31.75" rot="R90"/>
+<element name="R8" library="rcl" package="0207/7" value="1k" x="48.26" y="31.75" rot="R90"/>
 <element name="R11" library="rcl" package="0207/7" value="10k" x="45.72" y="31.75" rot="R270"/>
 <element name="JP1" library="pinhead" package="1X04" value="Out-Value" x="60.96" y="31.75" rot="R90"/>

Commit message: VA-Meter_Analog_Part 回路図、基板図、電流値を一つにまとめてGND値を出力するように変更 アナログ部テスト 更新
Connections:
- net A-M renamed IM
- net GND+ renamed NC
- net GND- renamed GIN
- removed net A+M: IC2.1, JP1.2, R7.2
- new net N$1: IC2.1, R7.2
- net GND: now also JP1.2
Routing:
- net A+M: track 24.4 -> 0.00 mm
- net GND: track 177.8 -> 185.4 mm
Changed lines of the file:
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@@
 <contactref element="C2" pad="1"/>
 <wire x1="48.26" y1="35.56" x2="53.34" y2="35.56" width="0.4064" layer="16"/>
-<wire x1="53.34" y1="35.56" x2="53.34" y2="22.86" width="0.4064" layer="16"/>
+<wire x1="53.34" y1="35.56" x2="53.34" y2="30.48" width="0.4064" layer="16"/>
+<wire x1="53.34" y1="30.48" x2="53.34" y2="22.86" width="0.4064" layer="16"/>
 <wire x1="40.64" y1="20.32" x2="40.64" y2="5.08" width="0.4064" layer="16"/>
 <wire x1="40.64" y1="5.08" x2="45.72" y2="5.08" width="0.4064" layer="16"/>
@@
 <wire x1="63.5" y1="22.86" x2="63.5" y2="7.62" width="0.4064" layer="16"/>
 <wire x1="63.5" y1="7.62" x2="45.72" y2="7.62" width="0.4064" layer="16"/>
-<wire x1="7.493" y1="22.86" x2="5.08" y2="22.86" width="0" layer="19" extent="16-16"/>
 <wire x1="40.64" y1="20.32" x2="38.1" y2="20.32" width="0.4064" layer="16"/>
 <wire x1="38.1" y1="20.32" x2="38.1" y2="33.02" width="0.4064" layer="16"/>
@@
 <wire x1="30.48" y1="33.02" x2="30.48" y2="22.86" width="0.4064" layer="16"/>
 <wire x1="30.48" y1="22.86" x2="15.24" y2="22.86" width="0.4064" layer="16"/>
+<contactref element="JP1" pad="2"/>
+<wire x1="60.96" y1="30.48" x2="53.34" y2="30.48" width="0.4064" layer="16"/>
+<wire x1="5.08" y1="22.86" x2="7.493" y2="22.86" width="0" layer="19" extent="16-16"/>
 </signal>
 <signal name="MEAS-">
@@
 <wire x1="63.5" y1="33.02" x2="60.96" y2="33.02" width="0.4064" layer="16"/>
 </signal>
-<signal name="GND+">
+<signal name="NC">
 <contactref element="R5" pad="2"/>
 <contactref element="GND" pad="1"/>
@@
 <wire x1="48.26" y1="17.78" x2="30.48" y2="12.7" width="0.4064" layer="1"/>
 </signal>
-<signal name="GND-">
+<signal name="GIN">
 <contactref element="R6" pad="2"/>
 <contactref element="GND" pad="2"/>
@@
 <wire x1="45.72" y1="35.56" x2="48.26" y2="27.94" width="0.4064" layer="16"/>
 </signal>
-<signal name="A+M">
-<contactref element="R7" pad="2"/>
-<contactref element="IC2" pad="1"/>
-<contactref element="JP1" pad="2"/>
-<wire x1="43.18" y1="17.78" x2="43.18" y2="15.24" width="0.4064" layer="16"/>
-<wire x1="43.18" y1="17.78" x2="60.96" y2="30.48" width="0.4064" layer="1"/>
-</signal>
-<signal name="A-M">
+<signal name="IM">
 <contactref element="IC2" pad="7"/>
 <contactref element="R11" pad="2"/>
@@
 <wire x1="45.72" y1="27.94" x2="60.96" y2="35.56" width="0.4064" layer="1"/>
 </signal>
+<signal name="N$1">
+<contactref element="IC2" pad="1"/>
+<contactref element="R7" pad="2"/>
+<wire x1="43.18" y1="15.24" x2="43.18" y2="17.78" width="0" layer="19" extent="1-1"/>
+</signal>
 </signals>
