File: eagle/VA-Meter_Analog_Part.sch (EAGLE design)
At the start: 17 parts, among them IC2 LM358N

Commit message: アナログ部の修正 電流値の増幅を11倍に変更
Parts:
- R2, R8: value 2k -> 1k
Changed lines of the file:
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@@
 <?xml version="1.0" encoding="utf-8"?>
 <!DOCTYPE eagle SYSTEM "eagle.dtd">
-<eagle version="6.6.0">
+<eagle version="7.1.0">
 <drawing>
 <settings>
@@
 <setting verticaltext="up"/>
 </settings>
-<grid distance="0.1" unitdist="inch" unit="inch" style="dots" multiple="1" display="yes" altdistance="0.01" altunitdist="inch" altunit="inch"/>
+<grid distance="0.1" unitdist="inch" unit="inch" style="lines" multiple="1" display="no" altdistance="0.01" altunitdist="inch" altunit="inch"/>
 <layers>
 <layer number="1" name="Top" color="4" fill="1" visible="no" active="no"/>
@@
 <part name="P+4" library="supply1" deviceset="V+" device=""/>
 <part name="IC2" library="linear" deviceset="LM358" device="N"/>
-<part name="R2" library="rcl" deviceset="R-EU_" device="0207/7" value="2k"/>
+<part name="R2" library="rcl" deviceset="R-EU_" device="0207/7" value="1k"/>
 <part name="R7" library="rcl" deviceset="R-EU_" device="0207/7" value="10k"/>
 <part name="SUPPLY4" library="supply2" deviceset="GND" device=""/>
-<part name="R8" library="rcl" deviceset="R-EU_" device="0207/7" value="2k"/>
+<part name="R8" library="rcl" deviceset="R-EU_" device="0207/7" value="1k"/>
 <part name="R11" library="rcl" deviceset="R-EU_" device="0207/7" value="10k"/>
 <part name="SUPPLY6" library="supply2" deviceset="GND" device=""/>

Commit message: VA-Meter_Analog_Part 回路図、基板図、電流値を一つにまとめてGND値を出力するように変更 アナログ部テスト 更新
Connections:
- net A-M renamed IM
- net GND+ renamed NC
- net GND- renamed GIN
- removed net A+M: IC2A.OUT, JP1.2, R7.2
- new net N$1: IC2A.OUT, R7.2
- net GND: now also JP1.2
Changed lines of the file:
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@@
 <setting verticaltext="up"/>
 </settings>
-<grid distance="0.1" unitdist="inch" unit="inch" style="lines" multiple="1" display="no" altdistance="0.01" altunitdist="inch" altunit="inch"/>
+<grid distance="0.1" unitdist="inch" unit="inch" style="dots" multiple="1" display="yes" altdistance="0.01" altunitdist="inch" altunit="inch"/>
 <layers>
 <layer number="1" name="Top" color="4" fill="1" visible="no" active="no"/>
@@
 <part name="P+1" library="supply1" deviceset="V+" device=""/>
 <part name="P-2" library="supply1" deviceset="V-" device=""/>
+<part name="SUPPLY8" library="supply2" deviceset="GND" device=""/>
 </parts>
 <sheets>
@@
 <attribute name="VALUE" x="181.102" y="68.58" size="1.778" layer="96"/>
 </instance>
+<instance part="SUPPLY8" gate="GND" x="170.18" y="119.38"/>
 </instances>
 <busses>
@@
 <wire x1="195.58" y1="83.82" x2="185.42" y2="83.82" width="0.1524" layer="91"/>
 <junction x="185.42" y="83.82"/>
+</segment>
+<segment>
+<pinref part="SUPPLY8" gate="GND" pin="GND"/>
+<wire x1="170.18" y1="121.92" x2="170.18" y2="129.54" width="0.1524" layer="91"/>
+<pinref part="JP1" gate="A" pin="2"/>
+<wire x1="170.18" y1="129.54" x2="187.96" y2="129.54" width="0.1524" layer="91"/>
 </segment>
 </net>
@@
 </segment>
 </net>
-<net name="GND+" class="0">
+<net name="NC" class="0">
 <segment>
 <pinref part="R5" gate="G$1" pin="2"/>
@@
 </segment>
 </net>
-<net name="GND-" class="0">
+<net name="GIN" class="0">
 <segment>
 <pinref part="R6" gate="G$1" pin="2"/>
@@
 </segment>
 </net>
-<net name="A+M" class="0">
-<segment>
-<wire x1="152.4" y1="129.54" x2="152.4" y2="86.36" width="0.1524" layer="91"/>
-<wire x1="152.4" y1="86.36" x2="152.4" y2="76.2" width="0.1524" layer="91"/>
-<wire x1="152.4" y1="129.54" x2="187.96" y2="129.54" width="0.1524" layer="91"/>
-<pinref part="R7" gate="G$1" pin="2"/>
-<wire x1="142.24" y1="76.2" x2="152.4" y2="76.2" width="0.1524" layer="91"/>
-<pinref part="IC2" gate="A" pin="OUT"/>
-<wire x1="147.32" y1="86.36" x2="152.4" y2="86.36" width="0.1524" layer="91"/>
-<junction x="152.4" y="86.36"/>
-<pinref part="JP1" gate="A" pin="2"/>
-<label x="175.26" y="129.54" size="1.778" layer="95"/>
-</segment>
-</net>
-<net name="A-M" class="0">
+<net name="IM" class="0">
 <segment>
 <wire x1="157.48" y1="60.96" x2="157.48" y2="124.46" width="0.1524" layer="91"/>
@@
 </segment>
 </net>
+<net name="N$1" class="0">
+<segment>
+<pinref part="IC2" gate="A" pin="OUT"/>
+<wire x1="147.32" y1="86.36" x2="152.4" y2="86.36" width="0.1524" layer="91"/>
+<wire x1="152.4" y1="86.36" x2="152.4" y2="76.2" width="0.1524" layer="91"/>
+<pinref part="R7" gate="G$1" pin="2"/>
+<wire x1="142.24" y1="76.2" x2="152.4" y2="76.2" width="0.1524" layer="91"/>
+</segment>
+</net>
