File: eagle/VA-Meter_Measure.brd (EAGLE design)
At the start: 100 x 80 mm, 10 parts, among them IC1 MEGA328P

Commit message: VA-Meter_Measure 回路図、SCLとSDAの信号線の名前が逆だったのを修正
Connections:
- net SCL: now also IC1.28, JP1.4; no longer IC1.27, JP1.3
- net SDA: now also IC1.27, JP1.3; no longer IC1.28, JP1.4
Changed lines of the file:
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@@
 <wire x1="50.76" y1="25.4" x2="58.42" y2="25.4" width="0.4064" layer="16"/>
 </signal>
-<signal name="SCL">
+<signal name="SDA">
 <contactref element="IC1" pad="27"/>
 <contactref element="JP1" pad="3"/>
 <wire x1="20.32" y1="38.1" x2="20.32" y2="17.78" width="0.4064" layer="16"/>
 </signal>
-<signal name="SDA">
+<signal name="SCL">
 <contactref element="IC1" pad="28"/>
 <contactref element="JP1" pad="4"/>

Commit message: VA-Meter_Measure 電流電圧計デジタル部基板図修正
Parts:
- moved R4 2.54 mm to (10.2, 29.2)
- moved JP3 2.54 mm to (11.4, 38.1)
Routing:
- net V-: track 84.0 -> 81.5 mm
- net V+: track 109.3 -> 106.7 mm
Changed lines of the file:
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@@
 <?xml version="1.0" encoding="utf-8"?>
 <!DOCTYPE eagle SYSTEM "eagle.dtd">
-<eagle version="6.6.0">
+<eagle version="7.1.0">
 <drawing>
 <settings>
@@
 <layer number="98" name="Guide" color="6" fill="1" visible="no" active="no"/>
 <layer number="99" name="SpiceOrder" color="5" fill="1" visible="no" active="no"/>
-<layer number="100" name="Mesh" color="7" fill="1" visible="yes" active="yes"/>
+<layer number="100" name="Mesh" color="7" fill="1" visible="no" active="yes"/>
 <layer number="101" name="Grid" color="7" fill="1" visible="no" active="yes"/>
 </layers>
@@
 <pass name="Default">
 <param name="RoutingGrid" value="50mil"/>
+<param name="AutoGrid" value="1"/>
+<param name="Efforts" value="0"/>
+<param name="TopRouterVariant" value="1"/>
 <param name="tpViaShape" value="round"/>
 <param name="PrefDir.1" value="|"/>
@@
 <element name="L1" library="rcl" package="6000-XXXX-RC" value="10uH" x="48.26" y="25.4"/>
 <element name="C4" library="rcl" package="C050-024X044" value="0.1u" x="35.56" y="7.62"/>
-<element name="JP3" library="pinhead" package="1X02" value="LCD-BL" x="8.89" y="38.1" rot="R180"/>
-<element name="R4" library="rcl" package="0207/7" value="470" x="7.62" y="29.21" rot="R270"/>
+<element name="JP3" library="pinhead" package="1X02" value="LCD-BL" x="11.43" y="38.1" rot="R180"/>
+<element name="R4" library="rcl" package="0207/7" value="470" x="10.16" y="29.21" rot="R270"/>
 <element name="C5" library="rcl" package="C050-024X044" value="0.1u" x="35.56" y="22.86"/>
 <element name="JP1" library="pinhead" package="1X05" value="I2C-LCD" x="20.32" y="38.1" rot="R180"/>
@@
 <contactref element="JP3" pad="1"/>
 <contactref element="JP4" pad="3"/>
-<wire x1="10.16" y1="38.1" x2="10.16" y2="40.64" width="0.4064" layer="16"/>
-<wire x1="10.16" y1="40.64" x2="22.86" y2="40.64" width="0.4064" layer="16"/>
+<wire x1="12.7" y1="38.1" x2="12.7" y2="40.64" width="0.4064" layer="16"/>
+<wire x1="12.7" y1="40.64" x2="22.86" y2="40.64" width="0.4064" layer="16"/>
 <wire x1="22.86" y1="40.64" x2="22.86" y2="38.1" width="0.4064" layer="16"/>
 <wire x1="38.1" y1="7.62" x2="35.56" y2="7.62" width="0.4064" layer="16"/>
@@
 <contactref element="R4" pad="2"/>
 <contactref element="JP4" pad="1"/>
-<wire x1="7.62" y1="25.4" x2="7.62" y2="5.08" width="0.4064" layer="16"/>
-<wire x1="7.62" y1="5.08" x2="33.02" y2="5.08" width="0.4064" layer="16"/>
+<wire x1="10.16" y1="25.4" x2="10.16" y2="5.08" width="0.4064" layer="16"/>
+<wire x1="10.16" y1="5.08" x2="33.02" y2="5.08" width="0.4064" layer="16"/>
 <wire x1="33.02" y1="5.08" x2="33.02" y2="7.62" width="0.4064" layer="16"/>
 <wire x1="33.02" y1="10.16" x2="33.02" y2="7.62" width="0.4064" layer="16"/>
@@
 <contactref element="JP3" pad="2"/>
 <contactref element="R4" pad="1"/>
-<wire x1="7.62" y1="38.1" x2="7.62" y2="33.02" width="0.4064" layer="16"/>
+<wire x1="10.16" y1="38.1" x2="10.16" y2="33.02" width="0.4064" layer="16"/>
 </signal>
 <signal name="N$9">

Commit message: VA-Meter_Measure.sch デジタル部回路図修正 入力端子名の変更
Connections:
- net A+MEAS renamed G_MEAS
- net A-MEAS renamed I_MEAS
Changed lines of the file:
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@@
 <wire x1="38.1" y1="27.94" x2="38.1" y2="38.1" width="0.4064" layer="16"/>
 </signal>
-<signal name="A+MEAS">
+<signal name="G_MEAS">
 <contactref element="JP2" pad="2"/>
 <contactref element="IC1" pad="24"/>
@@
 <wire x1="33.02" y1="33.02" x2="33.02" y2="38.1" width="0.4064" layer="16"/>
 </signal>
-<signal name="A-MEAS">
+<signal name="I_MEAS">
 <contactref element="IC1" pad="26"/>
 <contactref element="JP2" pad="4"/>
